File: build/DCLK-MIDI-Clock/DCLK-MIDI-Clock.kicad_sch (KiCad schematic)
At the start: 44 parts, among them J1 MIDI OUT, J2 Jack-DC, J3 MIDI OUT, J5 Conn_02x04_Odd_Even, J6 Conn_02x04_Odd_Even, J7 SYNC 1 OUT, J8 SYNC 2 OUT, SW4 RotaryEncoder_Switch_MP, U2 CAP1206-x-SL, U3 74AHCT125

Commit message: symbol fields update
Parts:
- R1, R10, R2, R3, R4, R5, R6, R7, R8, R9: Part Number RT0402FRE0710KL -> (none); Part Number 2 RT0402DRE0710KL -> (none)
Changed lines of the file:
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@@
 			)
 		)
-		(property "Part Number" "RT0402FRE0710KL"
+		(property "Part Number" ""
 			(at 82.55 98.298 0)
 			(effects
@@
 			)
 		)
-		(property "Part Number 2" "RT0402DRE0710KL"
+		(property "Part Number 2" ""
 			(at 80.01 109.22 0)
 			(effects
@@
 			)
 		)
-		(property "Part Number" "RT0402FRE0710KL"
+		(property "Part Number" ""
 			(at 167.64 113.792 0)
 			(effects
@@
 			)
 		)
-		(property "Part Number 2" "RT0402DRE0710KL"
+		(property "Part Number 2" ""
 			(at 170.18 102.87 0)
 			(effects
@@
 			)
 		)
-		(property "Part Number" "RT0402FRE0710KL"
+		(property "Part Number" ""
 			(at 119.38 112.522 0)
 			(effects
@@
 			)
 		)
-		(property "Part Number 2" "RT0402DRE0710KL"
+		(property "Part Number 2" ""
 			(at 121.92 101.6 0)
 			(effects
@@
 			)
 		)
-		(property "Part Number" "RT0402FRE0710KL"
+		(property "Part Number" ""
 			(at 38.1 98.298 0)
 			(effects
@@
 			)
 		)
-		(property "Part Number 2" "RT0402DRE0710KL"
+		(property "Part Number 2" ""
 			(at 35.56 109.22 0)
 			(effects
@@
 			)
 		)
-		(property "Part Number" "RT0402FRE0710KL"
+		(property "Part Number" ""
 			(at 115.57 112.522 0)
 			(effects
@@
 			)
 		)
-		(property "Part Number 2" "RT0402DRE0710KL"
+		(property "Part Number 2" ""
 			(at 118.11 101.6 0)
 			(effects
@@
 			)
 		)
-		(property "Part Number" "RT0402FRE0710KL"
+		(property "Part Number" ""
 			(at 180.34 113.792 0)
 			(effects
@@
 			)
 		)
-		(property "Part Number 2" "RT0402DRE0710KL"
+		(property "Part Number 2" ""
 			(at 182.88 102.87 0)
 			(effects
@@
 			)
 		)
-		(property "Part Number" "RT0402FRE0710KL"
+		(property "Part Number" ""
 			(at 86.36 98.298 0)
 			(effects
@@
 			)
 		)
-		(property "Part Number 2" "RT0402DRE0710KL"
+		(property "Part Number 2" ""
 			(at 83.82 109.22 0)
 			(effects
@@
 			)
 		)
-		(property "Part Number" "RT0402FRE0710KL"
+		(property "Part Number" ""
 			(at 198.12 85.852 0)
 			(effects
@@
 			)
 		)
-		(property "Part Number 2" "RT0402DRE0710KL"
+		(property "Part Number 2" ""
 			(at 200.66 74.93 0)
 			(effects
@@
 			)
 		)
-		(property "Part Number" "RT0402FRE0710KL"
+		(property "Part Number" ""
 			(at 41.91 98.298 0)
 			(effects
@@
 			)
 		)
-		(property "Part Number 2" "RT0402DRE0710KL"
+		(property "Part Number 2" ""
 			(at 39.37 109.22 0)
 			(effects
@@
 			)
 		)
-		(property "Part Number" "RT0402FRE0710KL"
+		(property "Part Number" ""
 			(at 158.75 113.792 0)
 			(effects
@@
 			)
 		)
-		(property "Part Number 2" "RT0402DRE0710KL"
+		(property "Part Number 2" ""
 			(at 161.29 102.87 0)
 			(effects
