File: build/DCLK-MIDI-Clock/DCLK-MIDI-Clock.kicad_sch (KiCad schematic)
At the start: 44 parts, among them J1 MIDI OUT, J2 Jack-DC, J3 MIDI OUT, J5 Conn_02x04_Odd_Even, J6 Conn_02x04_Odd_Even, J7 SYNC 1 OUT, J8 SYNC 2 OUT, SW4 RotaryEncoder_Switch_MP, U2 CAP1206-x-SL, U3 74AHCT125

Commit message: symbol fields
Parts:
- C1, C6: JLCPCB ID C14663 -> (none); Part Number 0603YC104KAT2A -> (none)
Changed lines of the file:
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@@
 			)
 		)
-		(property "Part Number" "0603YC104KAT2A"
+		(property "Part Number" ""
 			(at 120.65 104.648 0)
 			(effects
@@
 			)
 		)
-		(property "JLCPCB ID" "C14663"
+		(property "JLCPCB ID" ""
 			(at 116.84 102.87 0)
 			(effects
@@
 			)
 		)
-		(property "Part Number" "0603YC104KAT2A"
+		(property "Part Number" ""
 			(at 127 19.558 0)
 			(effects
@@
 			)
 		)
-		(property "JLCPCB ID" "C14663"
+		(property "JLCPCB ID" ""
 			(at 123.19 17.78 0)
 			(effects
