File: build/DCLK-MIDI-Clock/DCLK-MIDI-Clock.kicad_sch (KiCad schematic)
At the start: 44 parts, among them J1 MIDI OUT, J2 Jack-DC, J3 MIDI OUT, J5 Conn_02x04_Odd_Even, J6 Conn_02x04_Odd_Even, J7 SYNC 1 OUT, J8 SYNC 2 OUT, SW4 RotaryEncoder_Switch_MP, U2 CAP1206-x-SL, U3 74AHCT125

Commit message: Remove stale 0603 part fields from C1/C6 (now 1206)
Drops Part Number 0603YC104KAT2A, JLCPCB ID C14663 and Manufacturer AVX.

Co-Authored-By: Claude Opus 5.5 <noreply@anthropic.com>
Claude-Session: https://claude.ai/code/session_01XGX6wcyehYks8dMCrphrdY
Parts:
- C1, C6: JLCPCB ID C14663 -> (none); Manufacturer AVX Corporation -> (none); Part Number 0603YC104KAT2A -> (none)
Changed lines of the file:
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@@
-			)
-		)
-		(property "Manufacturer" "AVX Corporation"
-			(at 120.65 106.172 0)
-			(effects
-				(font
-					(size 1.27 1.27)
-				)
-				(justify left)
-				(hide yes)
-			)
-		)
-		(property "Part Number" "0603YC104KAT2A"
-			(at 120.65 104.648 0)
-			(effects
-				(font
-					(size 1.27 1.27)
-				)
-				(justify left)
-				(hide yes)
 			)
 		)
@@
 				)
 				(justify right)
-			)
-		)
-		(property "JLCPCB ID" "C14663"
-			(at 116.84 102.87 0)
-			(effects
-				(font
-					(size 1.27 1.27)
-				)
-				(hide yes)
 			)
 		)
@@
 			)
 		)
-		(property "Manufacturer" "AVX Corporation"
-			(at 127 21.082 0)
-			(effects
-				(font
-					(size 1.27 1.27)
-				)
-				(justify left)
-				(hide yes)
-			)
-		)
-		(property "Part Number" "0603YC104KAT2A"
-			(at 127 19.558 0)
-			(effects
-				(font
-					(size 1.27 1.27)
-				)
-				(justify left)
-				(hide yes)
-			)
-		)
 		(property "Display" "0.1uF"
 			(at 127 31.7435 0)
@@
 			)
 		)
-		(property "JLCPCB ID" "C14663"
-			(at 123.19 17.78 0)
-			(effects
-				(font
-					(size 1.27 1.27)
-				)
-				(hide yes)
-			)
-		)

Commit message: Add LCSC part numbers; clean C1/C6 footprint fields; remove J5 pin 7-8 track
- 'LCSC Part #' field on all 32 JLC-assembled parts (schematic + PCB),
  numbers taken from DCLK_bom_jcl.xls; 100nF (C1/C3/C6/C10) = C24497 (1206)
- Drop stale 0603 Part Number / JLCPCB ID / Manufacturer from C1/C6 footprints
- Delete stray track shorting unused J5 pins 7 and 8
- DCLK_bom.csv: LCSC column filled, mouse-bite tab row removed
- DCLK_bom_jcl.xls: 100nF line labelled 1206

Co-Authored-By: Claude Opus 5.5 <noreply@anthropic.com>
Claude-Session: https://claude.ai/code/session_01XGX6wcyehYks8dMCrphrdY
Parts:
- C1, C10, C3, C6: LCSC Part # (none) -> C24497
- C2, C4: LCSC Part # (none) -> C13585
- C7, C8, C9: LCSC Part # (none) -> C1846
- D1: LCSC Part # (none) -> C19167
- J5: LCSC Part # (none) -> C54907661
- J6: LCSC Part # (none) -> C41397153
- R1, R2, R3, R4: LCSC Part # (none) -> C23140
- R10: LCSC Part # (none) -> C15401
- R11, R12, R13, R14: LCSC Part # (none) -> C25530
- R15, R16, R17, R18: LCSC Part # (none) -> C11702
- R5, R6: LCSC Part # (none) -> C23162
- R7, R8, R9: LCSC Part # (none) -> C22104
- U2: LCSC Part # (none) -> C2652106
- U3: LCSC Part # (none) -> C155176
