File: build/DCLK-MIDI-Clock/DCLK-MIDI-Clock.kicad_pcb (KiCad board)
At the start: 2 copper layers, 125 x 213 mm, 76 parts, among them J1 MIDI OUT, J2 Jack-DC, J3 MIDI OUT, J5 Conn_02x04_Odd_Even, J6 Conn_02x04_Odd_Even, J7 SYNC 1 OUT, J8 SYNC 2 OUT, SW4 RotaryEncoder_Switch_MP, U2 CAP1206-x-SL, U3 74AHCT125

Commit message: Add LCSC part numbers; clean C1/C6 footprint fields; remove J5 pin 7-8 track
- 'LCSC Part #' field on all 32 JLC-assembled parts (schematic + PCB),
  numbers taken from DCLK_bom_jcl.xls; 100nF (C1/C3/C6/C10) = C24497 (1206)
- Drop stale 0603 Part Number / JLCPCB ID / Manufacturer from C1/C6 footprints
- Delete stray track shorting unused J5 pins 7 and 8
- DCLK_bom.csv: LCSC column filled, mouse-bite tab row removed
- DCLK_bom_jcl.xls: 100nF line labelled 1206

Co-Authored-By: Claude Opus 5.5 <noreply@anthropic.com>
Claude-Session: https://claude.ai/code/session_01XGX6wcyehYks8dMCrphrdY
Routing:
- net unconnected-(J5-Pin_8-Pad8): track 1.96 -> 0.00 mm
